File: 6502 Computer.kicad_sch (KiCad schematic)
At the start: 7 parts, among them SW1 CK_KMS2xxG, U1 6502, U2 MK4164N, U3 PL611-01-xxxT, U4 2764, U5 6522, U6 LCD-016N002L

Commit message: fixed issue with schematics where the wrong CPU was used <:(
Parts:
- removed SW1: CK_KMS2xxG, Button_Switch_SMD:SW_SPST_CK_KMS2xxGP, symbol Switch:CK_KMS2xxG
- removed U1: 6502, Package_DIP:DIP-40_W15.24mm, symbol 65xx-library:6502
- removed U2: MK4164N, Package_DIP:DIP-16_W7.62mm, symbol Memory_RAM:MK4164N
- removed U3: PL611-01-xxxT, Package_TO_SOT_SMD:SOT-23-6, symbol Timer:PL611-01-xxxT
- removed U4: 2764, Package_DIP:DIP-28_W15.24mm, symbol Memory_EPROM:2764
- removed U5: 6522, Package_DIP:DIP-40_W15.24mm, symbol 65xx-library:6522
- removed U6: LCD-016N002L, Display:LCD-016N002L, symbol Display_Character:LCD-016N002L
- added U1: W65C816SxP, Package_DIP:DIP-40_W15.24mm, symbol 65xx-library:W65C816SxP
- added U2: W65C22NxP, Package_DIP:DIP-40_W15.24mm, symbol 65xx-library:W65C22NxP
Connections:
- net +5V: now also U1.8 (VDD), U2.20 (VCC)
- net GND: now also U1.21 (VSS), U2.1 (VSS)
- new net: U1.26 (D7), U2.26 (D7)
- new net: U1.27 (D6), U2.27 (D6)
- new net: U1.28 (D5), U2.28 (D5)
- new net: U1.29 (D4), U2.29 (D4)
- new net: U1.30 (D3), U2.30 (D3)
- new net: U1.31 (D2), U2.31 (D2)
- new net: U1.32 (D1), U2.32 (D1)
- new net: U1.33 (D0), U2.33 (D0)
