File: clock.kicad_sch (KiCad schematic)
At the start: 1 part, among them U2 W65C22NxP

Commit message: Finished the EEPROM programmer and sent it off to get manufactured
Parts:
- removed U2: W65C22NxP, Package_DIP:DIP-40_W15.24mm, symbol 65xx-library:W65C22NxP
